Commit message: Gazebo Simulation

File: description/robot.urdf.xacro (robot description, xacro)
@@ -1,4 +1,5 @@
 <?xml version="1.0"?>
 <robot xmlns:xacro="http://www.ros.org/wiki/xacro"  name="robot">
-    <xacro:include filename="/home/thanhtan/ros_ws/src/my_bot/description/robot_core.xacro" />
+    <xacro:include filename="/home/thanhtan/ros_ws/src/my_bot/description/robot_core.xacro" /> <!--Tệp mô tả tổng quan hình dạng, tính chất robot-->
+    <xacro:include filename="/home/thanhtan/ros_ws/src/my_bot/description/gazebo_control.xacro" /> <!-- Tệp điều khiển robot trong môi trường Gazebo -->
 </robot>

File: description/robot_core.xacro (robot description, xacro)
@@ -46,12 +46,15 @@
          </xacro:inertial_box>
      </link>
-     <!-- Bánh xe Trái (LEFT WHELL LINK) tạo khớp động quay không giới hạn Continous -->
-     <joint name="left_whell_joint" type="continuous">
+     <gazebo reference="chassis">
+      <material>Gazebo/White</material>
+     </gazebo>
+     <!-- Bánh xe Trái (LEFT WHEEL LINK) tạo khớp động quay không giới hạn Continous -->
+     <joint name="left_wheel_joint" type="continuous">
       <parent link="base_link"/>
-      <child link="left_whell"/>
+      <child link="left_wheel"/>
       <origin xyz="0 0.105 0 " rpy="-${pi/2} 0 0"/>
       <axis xyz="0 0 1"/>
      </joint>
-     <link name="left_whell">
+     <link name="left_wheel">
       <visual>
          <geometry>
@@ -70,12 +73,15 @@
       </xacro:inertial_cylinder>
       </link>
-     <!-- BÁNH XE PHẢI (RIGHT WHELL LINK) -->
-     <joint name="right_whell_joint" type="continuous">
+      <gazebo reference="left_wheel">
+         <material>Gazebo/Blue</material>
+        </gazebo>
+     <!-- BÁNH XE PHẢI (RIGHT WHEEL LINK) -->
+     <joint name="right_wheel_joint" type="continuous">
       <parent link="base_link"/>
-      <child link="right_whell"/>
+      <child link="right_wheel"/>
       <origin xyz="0 -0.105 0 " rpy="${pi/2} 0 0"/>
       <axis xyz="0 0 -1"/>
      </joint>
-     <link name="right_whell">
+     <link name="right_wheel">
       <visual>
          <geometry>
@@ -94,11 +100,14 @@
        </xacro:inertial_cylinder>
       </link>
-      <!-- Bánh đa (CASTER WHELL LINK) -->
-      <joint name="caster_whell_link" type="fixed">
+      <gazebo reference="right_wheel">
+         <material>Gazebo/Blue</material>
+        </gazebo>
+      <!-- Bánh đa (CASTER WHEEL LINK) -->
+      <joint name="caster_wheel_link" type="fixed">
         <parent link="chassis"/>
-        <child link="caster_whell"/>
+        <child link="caster_wheel"/>
         <origin xyz="0.12 0 0"/>
       </joint>
-      <link name="caster_whell">
+      <link name="caster_wheel">
          <visual>
             <geometry>
@@ -117,3 +126,8 @@
          </xacro:inertial_sphere>
       </link>
+      <gazebo reference="caster_wheel">
+         <material>Gazebo/Black</material>
+         <mu1 value="0.001"/>
+         <mu2 value="0.001"/>
+        </gazebo>
 </robot>

Commit message: lindar va camera

File: description/robot.urdf.xacro (robot description, xacro)
@@ -3,3 +3,5 @@
     <xacro:include filename="/home/thanhtan/ros_ws/src/my_bot/description/robot_core.xacro" /> <!--Tệp mô tả tổng quan hình dạng, tính chất robot-->
     <xacro:include filename="/home/thanhtan/ros_ws/src/my_bot/description/gazebo_control.xacro" /> <!-- Tệp điều khiển robot trong môi trường Gazebo -->
+    <xacro:include filename="/home/thanhtan/ros_ws/src/my_bot/description/lidar.xacro" />
+    <xacro:include filename="/home/thanhtan/ros_ws/src/my_bot/description/camera.xacro" />
 </robot>

File: description/robot_core.xacro (robot description, xacro)
@@ -15,4 +15,7 @@
         <color rgba="0 0 0 1"/>
      </material>
+     <material name="red">
+      <color rgba="1 0 0 1"/>
+   </material>
      <!---->
      <!-- Kích thước tổng quan thân robot (0.18 x 0.13 x 0.5)(d x r x c)  m  có nghĩa là sẽ không có sự di chuyển giữa các liên kết nối với khớp này -->
